Commit message: update for rplidar

File: iRobot/iRobot.urdf (robot description, URDF)
Before this commit: robot iRobot, 9 links, 8 joints
Links:
- removed link hokuyo_laser_link
- added link laser, mass 1e-5; collision box size=0.1 0.1 0.1; visual cylinder length=0.1 radius=0.045
Joints:
- removed joint hokuyo_laser_joint
- added joint rplidar_laser_joint: type fixed, parent base_link, child laser, origin xyz=0.1 0 0.05 rpy=0 0 0, axis 0 0 1

File: model/iRobot.urdf.xacro (robot description, xacro)
@@ -7,5 +7,5 @@
   <xacro:include filename="$(find irobotcreate2)/model/shelf.urdf.xacro"/>
   <xacro:include filename="$(find irobotcreate2)/gazebo/iRobot.gazebo.xacro"/>
-  <xacro:include filename="$(find irobotcreate2)/model/hokuyo.urdf.xacro"/>
+  <xacro:include filename="$(find irobotcreate2)/model/rplidar.urdf.xacro"/>
   <xacro:property name="pi" value="3.1415926535897931"/>
   <xacro:property name="wheel_mass" value="0.5"/>
@@ -129,8 +129,8 @@
         </collision>
     </link>
-    <xacro:hokuyo_laser xyz="0 0 0.05"
+    <xacro:rplidar_laser xyz="0.1 0 0.05"
                   rpy="0 0 0"
                   parent="base_link">
-    </xacro:hokuyo_laser>
+    </xacro:rplidar_laser>
   <!--  <xacro:model_shelf name="first_shelf"
                        parent="chassis"

Commit message: update

File: iRobot/iRobot.urdf (robot description, URDF)
Before this commit: robot iRobot, 9 links, 8 joints
Joints:
- joint rplidar_laser_joint: origin xyz=0.1 0 0.05 rpy=0 0 0 -> xyz=-0.1 0 0.05 rpy=0 0 0

File: model/iRobot.urdf.xacro (robot description, xacro)
@@ -129,5 +129,5 @@
         </collision>
     </link>
-    <xacro:rplidar_laser xyz="0.1 0 0.05"
+    <xacro:rplidar_laser xyz="-0.1 0 0.05"
                   rpy="0 0 0"
                   parent="base_link">

Commit message: fix

File: iRobot/iRobot.urdf (robot description, URDF)
Before this commit: robot iRobot, 9 links, 8 joints
Joints:
- joint rplidar_laser_joint: origin xyz=-0.1 0 0.05 rpy=0 0 0 -> xyz=-0.1 0 0.05 rpy=0 0 1.57079632679

File: model/iRobot.urdf.xacro (robot description, xacro)
@@ -130,5 +130,5 @@
     </link>
     <xacro:rplidar_laser xyz="-0.1 0 0.05"
-                  rpy="0 0 0"
+                  rpy="0 0 ${pi/2}"
                   parent="base_link">
     </xacro:rplidar_laser>

Commit message: update

File: iRobot/iRobot.urdf (robot description, URDF)
Before this commit: robot iRobot, 9 links, 8 joints
Joints:
- joint rplidar_laser_joint: origin xyz=-0.1 0 0.05 rpy=0 0 1.57079632679 -> xyz=-0.1 0 0.05 rpy=0 3.14159265359 4.71238898038

File: model/iRobot.urdf.xacro (robot description, xacro)
@@ -130,5 +130,5 @@
     </link>
     <xacro:rplidar_laser xyz="-0.1 0 0.05"
-                  rpy="0 0 ${pi/2}"
+                  rpy="0 ${pi} ${pi/2+pi}"
                   parent="base_link">
     </xacro:rplidar_laser>
